File: Hardware/MicroMod_Processor_Board-nRF52840.brd (EAGLE design)
At the start: 22 x 22 mm, 28 parts, among them J2 MICROMOD-2222, U1 W25QXX128MBIT-6X5, U2 MDBT50Q, Y1 32.768kHz

Commit message: Preliminary schematic finished
Parts:
- added R4, R5: 10k, SparkFun-Resistors:0402-TIGHT
Connections:
- removed net 3.3V_EN: J2.4
- removed net BOOT: J2.11
- removed net N$6: U1.1
- new net !BOOT!: J2.11, R4.1, U2.37
- new net FLASH_!CS!: U1.1, U2.29
- net !RESET!: now also R5.1, U2.40
- net 3.3V: now also R4.2, R5.2
- net SPI_MOSI: now also U2.36; no longer U2.40
Changed lines of the file:
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@@
 </element>
 <element name="J2" library="SparkFun-MicroMod" package="M.2-CARD-E-22" value="MICROMOD-2222" x="10.922" y="0" smashed="yes"/>
+<element name="R4" library="SparkFun-Resistors" package="0402-TIGHT" value="10k" x="-55.88" y="-43.18" smashed="yes">
+<attribute name="NAME" x="-55.88" y="-42.618" size="0.6096" layer="25" font="vector" ratio="20" align="bottom-center"/>
+<attribute name="PROD_ID" value="RES-14241" x="-55.88" y="-43.18" size="1.778" layer="27" font="vector" ratio="15" display="off"/>
+<attribute name="VALUE" x="-55.88" y="-43.742" size="0.6096" layer="27" font="vector" ratio="20" align="top-center"/>
+</element>
+<element name="R5" library="SparkFun-Resistors" package="0402-TIGHT" value="10k" x="-55.88" y="-46.99" smashed="yes">
+<attribute name="NAME" x="-55.88" y="-46.428" size="0.6096" layer="25" font="vector" ratio="20" align="bottom-center"/>
+<attribute name="PROD_ID" value="RES-14241" x="-55.88" y="-46.99" size="1.778" layer="27" font="vector" ratio="15" display="off"/>
+<attribute name="VALUE" x="-55.88" y="-47.552" size="0.6096" layer="27" font="vector" ratio="20" align="top-center"/>
+</element>
 </elements>
 <signals>
@@
 <contactref element="J2" pad="74"/>
 <contactref element="J2" pad="2"/>
-<wire x1="19.922" y1="1.525" x2="1.922" y2="1.525" width="0" layer="19" extent="16-16"/>
-<wire x1="-56.38" y1="-35.56" x2="19.922" y2="1.525" width="0" layer="19" extent="1-16"/>
-<wire x1="-56.46" y1="-39.37" x2="-56.38" y2="-35.56" width="0" layer="19" extent="1-1"/>
+<contactref element="R4" pad="2"/>
+<contactref element="R5" pad="2"/>
+<wire x1="-55.38" y1="-43.18" x2="-55.38" y2="-46.99" width="0" layer="19" extent="1-1"/>
+<wire x1="-56.46" y1="-39.37" x2="-55.38" y2="-43.18" width="0" layer="19" extent="1-1"/>
+<wire x1="-56.38" y1="-35.56" x2="-56.46" y2="-39.37" width="0" layer="19" extent="1-1"/>
 <wire x1="-56.38" y1="-31.75" x2="-56.38" y2="-35.56" width="0" layer="19" extent="1-1"/>
 <wire x1="-38.68" y1="-12.7" x2="-56.38" y2="-31.75" width="0" layer="19" extent="1-1"/>
 <wire x1="-31.515" y1="-3.175" x2="-38.68" y2="-12.7" width="0" layer="19" extent="1-1"/>
-<wire x1="18.68" y1="13.03" x2="-31.515" y2="-3.175" width="0" layer="19" extent="1-1"/>
+<wire x1="1.922" y1="1.525" x2="-31.515" y2="-3.175" width="0" layer="19" extent="1-16"/>
+<wire x1="19.922" y1="1.525" x2="1.922" y2="1.525" width="0" layer="19" extent="16-16"/>
+<wire x1="18.68" y1="13.03" x2="19.922" y2="1.525" width="0" layer="19" extent="1-16"/>
 <wire x1="18.68" y1="13.83" x2="18.68" y2="13.03" width="0" layer="19" extent="1-1"/>
 </signal>
@@
 <signal name="SPI_MOSI">
 <contactref element="J2" pad="62"/>
-<contactref element="U2" pad="40"/>
-<wire x1="14.88" y1="15.18" x2="4.922" y2="1.525" width="0" layer="19" extent="1-16"/>
+<contactref element="U2" pad="36"/>
+<wire x1="4.922" y1="1.525" x2="16.48" y2="15.18" width="0" layer="19" extent="1-16"/>
 </signal>
 <signal name="SPI_!CS!">
@@
 <wire x1="14.922" y1="1.525" x2="12.08" y2="11.03" width="0" layer="19" extent="1-16"/>
 </signal>
-<signal name="N$6">
+<signal name="FLASH_!CS!">
 <contactref element="U1" pad="1"/>
+<contactref element="U2" pad="29"/>
+<wire x1="17.78" y1="13.43" x2="-37.065" y2="-3.175" width="0" layer="19" extent="1-1"/>
 </signal>
 <signal name="USB_VIN">
@@
 <signal name="!RESET!">
 <contactref element="J2" pad="6"/>
-</signal>
-<signal name="BOOT">
+<contactref element="U2" pad="40"/>
+<contactref element="R5" pad="1"/>
+<wire x1="18.922" y1="1.525" x2="-56.38" y2="-46.99" width="0" layer="19" extent="1-16"/>
+<wire x1="14.88" y1="15.18" x2="18.922" y2="1.525" width="0" layer="19" extent="1-16"/>
+</signal>
+<signal name="!BOOT!">
 <contactref element="J2" pad="11"/>
+<contactref element="U2" pad="37"/>
+<contactref element="R4" pad="1"/>
+<wire x1="17.672" y1="1.275" x2="-56.38" y2="-43.18" width="0" layer="19" extent="1-1"/>
+<wire x1="16.08" y1="16.08" x2="17.672" y2="1.275" width="0" layer="19" extent="1-1"/>
 </signal>
 <signal name="I2C_!INT!">
@@
 <wire x1="6.672" y1="1.275" x2="12.88" y2="16.08" width="0" layer="19" extent="1-1"/>
 </signal>
-<signal name="3.3V_EN">
-<contactref element="J2" pad="4"/>
-</signal>
 <signal name="RX2">

Commit message: Finished preliminary schematic
Parts:
- moved J2 0.08 mm to (11.0, 0.00)
Connections:
- net PDM_DATA: now also U2.19; no longer U2.50
- net RTS1: now also U2.50; no longer U2.19

Commit message: Preliminary layout of PB
Parts:
- moved R5 95.2 mm to (13.6, 18.0), turned to 90 degrees
- moved R4 93.4 mm to (14.6, 18.0), turned to 90 degrees
- moved C4 88.3 mm to (19.9, 13.6)
- moved C5 86.9 mm to (12.6, 18.0), turned to 270 degrees
- moved C2 84.3 mm to (20.3, 11.9), turned to 270 degrees
- moved C3 83.4 mm to (20.3, 5.84), turned to 90 degrees
- moved Y1 81.2 mm to (20.3, 8.89), turned to 90 degrees
- moved R3 80.0 mm to (19.1, 18.7), turned to 90 degrees
- moved R2 77.1 mm to (17.8, 18.7), turned to 270 degrees
- moved C6 73.2 mm to (1.27, 6.35), turned to 90 degrees
- moved C1 54.3 mm to (8.26, 15.5), flipped to the bottom, turned to 90 degrees
- moved U1 48.2 mm to (11.0, 11.4), flipped to the bottom
- moved U2 1.27 mm to (10.2, 11.4)
- moved FD1 0.54 mm to (0.62, 4.62)
Other:
- board text removed: "N. Seidle"
