File: Hardware/MicroMod_Processor_Board-nRF52840.brd (EAGLE design)
At the start: 22 x 22 mm, 30 parts, among them J2 MICROMOD-2222, U1 W25QXX128MBIT-6X5, U2 MDBT50Q, Y1 32.768kHz

Commit message: Routing
Parts:
- C2, C3, C6: device SparkFun-Capacitors:0402 -> SparkFun-Capacitors:0402-TIGHT
Changed lines of the file:
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@@
 <?xml version="1.0" encoding="utf-8"?>
 <!DOCTYPE eagle SYSTEM "eagle.dtd">
-<eagle version="9.4.2">
+<eagle version="9.5.2">
 <drawing>
 <settings>
-<setting alwaysvectorfont="yes"/>
+<setting alwaysvectorfont="no"/>
 <setting verticaltext="up"/>
 </settings>
@@
 <layer number="38" name="bTest" color="7" fill="1" visible="no" active="yes"/>
 <layer number="39" name="tKeepout" color="4" fill="11" visible="yes" active="yes"/>
-<layer number="40" name="bKeepout" color="1" fill="11" visible="no" active="yes"/>
-<layer number="41" name="tRestrict" color="4" fill="10" visible="no" active="yes"/>
-<layer number="42" name="bRestrict" color="1" fill="10" visible="no" active="yes"/>
+<layer number="40" name="bKeepout" color="1" fill="11" visible="yes" active="yes"/>
+<layer number="41" name="tRestrict" color="4" fill="10" visible="yes" active="yes"/>
+<layer number="42" name="bRestrict" color="1" fill="10" visible="yes" active="yes"/>
 <layer number="43" name="vRestrict" color="2" fill="10" visible="no" active="yes"/>
 <layer number="44" name="Drills" color="7" fill="1" visible="no" active="yes"/>
@@
 <layer number="47" name="Measures" color="7" fill="1" visible="no" active="yes"/>
 <layer number="48" name="Document" color="7" fill="1" visible="no" active="yes"/>
-<layer number="49" name="Reference" color="7" fill="1" visible="yes" active="yes"/>
+<layer number="49" name="Reference" color="7" fill="1" visible="no" active="yes"/>
 <layer number="50" name="dxf" color="7" fill="1" visible="no" active="yes"/>
 <layer number="51" name="tDocu" color="6" fill="1" visible="yes" active="yes"/>
@@
 <attribute name="VALUE" x="21.363" y="8.89" size="0.6096" layer="27" font="vector" ratio="20" rot="R90" align="top-center"/>
 </element>
-<element name="C2" library="SparkFun-Capacitors" package="0402" value="15pF" x="20.32" y="11.938" smashed="yes" rot="R270">
+<element name="C2" library="SparkFun-Capacitors" package="0402-TIGHT" value="15pF" x="20.32" y="11.938" smashed="yes" rot="R270">
 <attribute name="NAME" x="21.082" y="11.938" size="0.6096" layer="25" font="vector" ratio="20" rot="R270" align="bottom-center"/>
 <attribute name="PROD_ID" value="CAP-13063" x="20.32" y="11.938" size="1.778" layer="27" font="vector" ratio="15" rot="R270" display="off"/>
 <attribute name="VALUE" x="19.558" y="11.938" size="0.6096" layer="27" font="vector" ratio="20" rot="R270" align="top-center"/>
 </element>
-<element name="C3" library="SparkFun-Capacitors" package="0402" value="15pF" x="20.32" y="5.842" smashed="yes" rot="R90">
+<element name="C3" library="SparkFun-Capacitors" package="0402-TIGHT" value="15pF" x="20.32" y="5.842" smashed="yes" rot="R90">
 <attribute name="NAME" x="19.558" y="5.842" size="0.6096" layer="25" font="vector" ratio="20" rot="R90" align="bottom-center"/>
 <attribute name="PROD_ID" value="CAP-13063" x="20.32" y="5.842" size="1.778" layer="27" font="vector" ratio="15" rot="R90" display="off"/>
@@
 <attribute name="VALUE" x="12.011" y="18.034" size="0.6096" layer="27" font="vector" ratio="20" rot="R270" align="top-center"/>
 </element>
-<element name="C6" library="SparkFun-Capacitors" package="0402" value="0.1uF" x="1.27" y="6.35" smashed="yes" rot="R90">
+<element name="C6" library="SparkFun-Capacitors" package="0402-TIGHT" value="0.1uF" x="1.27" y="6.35" smashed="yes" rot="R90">
 <attribute name="NAME" x="0.508" y="6.35" size="0.6096" layer="25" font="vector" ratio="20" rot="R90" align="bottom-center"/>
 <attribute name="PROD_ID" value="CAP-12416" x="1.27" y="6.35" size="1.778" layer="27" font="vector" ratio="15" rot="R90" display="off"/>
@@
 <wire x1="2" y1="3.461" x2="1.27" y2="4.191" width="0.1016" layer="16"/>
 <via x="1.27" y="4.191" extent="1-16" drill="0.2032"/>
-<wire x1="1.27" y1="4.191" x2="1.27" y2="5.77" width="0.1016" layer="1"/>
+<wire x1="1.27" y1="4.191" x2="1.27" y2="5.85" width="0.1016" layer="1"/>
 <wire x1="8.225" y1="13.335" x2="8.255" y2="13.365" width="0.1016" layer="16"/>
 <wire x1="8.255" y1="13.365" x2="8.255" y2="14.914" width="0.1016" layer="16"/>
@@
 <wire x1="14.605" y1="18.534" x2="17.41" y2="13.83" width="0" layer="19" extent="1-1"/>
 <wire x1="8.255" y1="14.914" x2="12.573" y2="18.534" width="0" layer="19" extent="1-16"/>
-<wire x1="1.27" y1="5.77" x2="8.225" y2="13.335" width="0" layer="19" extent="1-16"/>
+<wire x1="1.27" y1="5.85" x2="8.225" y2="13.335" width="0" layer="19" extent="1-16"/>
 <wire x1="20" y1="1.525" x2="17.41" y2="13.03" width="0" layer="19" extent="1-16"/>
 </signal>
@@
 <contactref element="J2" pad="33"/>
 <contactref element="J2" pad="GND3"/>
-<wire x1="20.32" y1="12.518" x2="20.32" y2="12.954" width="0.1016" layer="1"/>
+<wire x1="20.32" y1="12.438" x2="20.32" y2="12.954" width="0.1016" layer="1"/>
 <wire x1="20.32" y1="12.954" x2="20.447" y2="13.081" width="0.1016" layer="1"/>
 <wire x1="20.447" y1="13.081" x2="20.447" y2="13.835" width="0.1016" layer="1"/>
 <wire x1="20.447" y1="13.835" x2="20.439" y2="13.843" width="0.1016" layer="1"/>
-<wire x1="15" y1="19.7" x2="17.1" y2="21" width="0" layer="19" extent="1-1"/>
-<wire x1="12.9" y1="21" x2="15" y2="19.7" width="0" layer="19" extent="1-1"/>
-<wire x1="12.573" y1="17.534" x2="15" y2="19.7" width="0" layer="19" extent="1-1"/>
-<wire x1="17.41" y1="16.23" x2="15" y2="19.7" width="0" layer="19" extent="1-1"/>
-<wire x1="20.439" y1="13.843" x2="17.41" y2="16.23" width="0" layer="19" extent="1-1"/>
-<wire x1="8.255" y1="16.074" x2="12.573" y2="17.534" width="0" layer="19" extent="1-16"/>
-<wire x1="6.51" y1="16.08" x2="8.255" y2="16.074" width="0" layer="19" extent="1-16"/>
-<wire x1="17.41" y1="6.63" x2="20.32" y2="12.518" width="0" layer="19" extent="1-1"/>
-<wire x1="20.32" y1="5.262" x2="17.41" y2="6.63" width="0" layer="19" extent="1-1"/>
-<wire x1="20.25" y1="1.275" x2="20.32" y2="5.262" width="0" layer="19" extent="1-1"/>
-<wire x1="18.75" y1="1.275" x2="20.25" y2="1.275" width="0" layer="19" extent="1-1"/>
-<wire x1="13.775" y1="9.525" x2="17.41" y2="6.63" width="0" layer="19" extent="1-16"/>
-<wire x1="12.25" y1="1.275" x2="18.75" y2="1.275" width="0" layer="19" extent="1-1"/>
-<wire x1="11.5" y1="1.525" x2="12.25" y2="1.275" width="0" layer="19" extent="1-16"/>
-<wire x1="10.75" y1="1.275" x2="11.5" y2="1.525" width="0" layer="19" extent="1-16"/>
 <wire x1="9.25" y1="1.275" x2="10.75" y2="1.275" width="0" layer="19" extent="1-1"/>
-<wire x1="7.61" y1="6.78" x2="9.25" y2="1.275" width="0" layer="19" extent="1-1"/>
-<wire x1="6.51" y1="6.78" x2="7.61" y2="6.78" width="0" layer="19" extent="1-1"/>
-<wire x1="1.27" y1="6.93" x2="6.51" y2="6.78" width="0" layer="19" extent="1-1"/>
-<wire x1="1.75" y1="1.275" x2="1.27" y2="6.93" width="0" layer="19" extent="1-1"/>
-<wire x1="2.123" y1="21" x2="6.51" y2="16.08" width="0" layer="19" extent="1-1"/>
 </signal>
 <signal name="SWDIO">
@@
 <wire x1="8.89" y1="11.303" x2="9.017" y2="11.43" width="0.1016" layer="2"/>
 <wire x1="14.732" y1="11.43" x2="9.017" y2="11.43" width="0.1016" layer="2"/>
-<wire x1="14.986" y1="11.684" x2="12.81" y2="15.18" width="0" layer="19" extent="1-1"/>
+<wire x1="14.986" y1="13.716" x2="12.81" y2="15.18" width="0" layer="19" extent="1-1"/>
 <wire x1="5.5" y1="1.525" x2="8.225" y2="10.795" width="0" layer="19" extent="16-16"/>
 </signal>
@@
 <wire x1="14.351" y1="10.033" x2="8.89" y2="10.033" width="0.1016" layer="2"/>
 <wire x1="12.01" y1="14.279" x2="12.446" y2="13.843" width="0.1016" layer="1"/>
-<wire x1="12.446" y1="13.843" x2="4.5" y2="1.525" width="0" layer="19" extent="16-16"/>
+<wire x1="4.5" y1="1.525" x2="8.225" y2="9.525" width="0" layer="19" extent="16-16"/>
 </signal>
 <signal name="SPI_MOSI">
@@
 <wire x1="20.3" y1="7.62" x2="20.32" y2="7.64" width="0.1016" layer="1"/>
 <wire x1="17.435" y1="8.255" x2="18.161" y2="8.255" width="0.1016" layer="1"/>
-<wire x1="20.32" y1="7.64" x2="20.32" y2="6.422" width="0.1016" layer="1"/>
+<wire x1="20.32" y1="7.64" x2="20.32" y2="6.342" width="0.1016" layer="1"/>
 </signal>
 <signal name="N$5">
@@
 <wire x1="18.923" y1="10.16" x2="20.3" y2="10.16" width="0.1016" layer="1"/>
 <wire x1="20.3" y1="10.16" x2="20.32" y2="10.14" width="0.1016" layer="1"/>
-<wire x1="20.32" y1="10.14" x2="20.32" y2="11.358" width="0.1016" layer="1"/>
+<wire x1="20.32" y1="10.14" x2="20.32" y2="11.438" width="0.1016" layer="1"/>
 </signal>
 <signal name="NFC1">

Commit message: Routing
Parts:
- C1: device SparkFun-Capacitors:0402 -> SparkFun-Capacitors:0402-TIGHT
- moved LOGO3 29.0 mm to (31.0, 21.0)
- moved U$1 27.5 mm to (28.1, 15.5)
- moved U$4 27.0 mm to (27.7, 18.8)
- moved U$3 26.0 mm to (27.1, 17.1)
- moved U$5 22.5 mm to (30.8, 7.40)
- moved LOGO1 21.5 mm to (31.0, 9.00)
- moved C6 21.5 mm to (20.6, 15.9), turned to 0 degrees
- moved LOGO2 16.2 mm to (35.0, 14.0)
- moved U$7 14.2 mm to (31.5, 14.9)
- moved C5 8.61 mm to (20.6, 14.9), turned to 0 degrees
- moved FD4 4.21 mm to (0.62, 4.62)
- moved R4 3.57 mm to (11.4, 19.7), turned to 180 degrees
- moved R5 2.25 mm to (11.4, 18.7), turned to 180 degrees
- moved R3 1.45 mm to (19.4, 18.7)
- moved R2 1.45 mm to (19.4, 20.3)
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Routing:
- net SPI_MOSI: track 0.00 -> 35.1 mm, vias 0 -> 1
- net SDIO_DATA2: track 6.67 -> 39.1 mm, vias 3 -> 4
- net SDIO_DATA1: track 7.00 -> 37.8 mm, vias 3 -> 5
- net SPI_MISO: track 13.8 -> 42.0 mm, vias 3 -> 5
- net SWDCK: track 22.4 -> 0.00 mm, vias 3 -> 0
- net RTS1: track 21.7 -> 0.03 mm, vias 3 -> 0
- net SWDIO: track 21.1 -> 0.03 mm, vias 3 -> 0
- net USB_D+: track 0.00 -> 21.0 mm, vias 0 -> 2
- net USB_D-: track 0.00 -> 19.2 mm, vias 0 -> 2
- net SPI_!CS!: track 18.9 -> 36.7 mm, vias 1 -> 3
- net SCL1: track 17.6 -> 0.00 mm, vias 3 -> 0
- net NFC2: track 17.4 -> 0.00 mm, vias 3 -> 0
- net PDM_CLK: track 17.1 -> 0.00 mm, vias 3 -> 0
- net I2C_!INT!: track 0.00 -> 16.9 mm, vias 0 -> 1
- net SDA1: track 0.00 -> 16.6 mm, vias 0 -> 2
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Other:
- board text added: "v10"
- board text removed: "v12"

Commit message: Routing
Connections:
- net ADC_D+: now also U2.10; no longer U2.13
- net ADC_D-: now also U2.9; no longer U2.11
- net BATT_VIN/3: now also U2.14; no longer U2.10
- net CTS1: now also U2.26; no longer U2.22
- net PWM0: now also U2.22; no longer U2.26
- net SPI_MISO1: now also U2.11; no longer U2.12
- net SPI_MOSI1: now also U2.12; no longer U2.9
- net SPI_SCK1: now also U2.13; no longer U2.14
Routing:
- net SPI_!CS!1: track 0.00 -> 33.4 mm, vias 0 -> 2
- net PDM_CLK: track 0.00 -> 31.7 mm, vias 0 -> 1
- net SCL1: track 0.00 -> 30.8 mm, vias 0 -> 2
- net PWM1: track 0.00 -> 21.5 mm, vias 0 -> 3
- net PDM_DATA: track 0.00 -> 18.5 mm, vias 0 -> 3
- net USB_VIN: track 0.00 -> 18.4 mm, vias 0 -> 2
- net NFC2: track 0.00 -> 15.9 mm, vias 0 -> 2
- net NFC1: track 0.00 -> 15.9 mm, vias 0 -> 2
- net ADC_D-: track 0.00 -> 14.7 mm
- net SPI_MISO1: track 0.00 -> 14.5 mm
- net SCL: track 0.00 -> 14.4 mm, vias 0 -> 1
- net CTS1: track 0.00 -> 14.0 mm, vias 0 -> 2
- net ADC1: track 0.00 -> 13.8 mm, vias 0 -> 1
- net ADC_D+: track 0.00 -> 13.7 mm
- net PWM0: track 0.00 -> 13.7 mm, vias 0 -> 1
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
Commit message: Routing
Parts:
- moved C1 1.83 mm to (8.12, 13.5), turned to 270 degrees
Connections:
- net RX1: now also U2.41; no longer U2.39
- net TX1: now also U2.39; no longer U2.41
Routing:
- net 3.3V: track 7.95 -> 55.0 mm, vias 0 -> 6
- net RTS1: track 0.00 -> 22.4 mm, vias 0 -> 3
- net SWDCK: track 0.00 -> 22.1 mm, vias 0 -> 3
- net SWDIO: track 0.03 -> 21.7 mm, vias 0 -> 3
- net !RESET!: track 4.57 -> 24.0 mm, vias 0 -> 3
- net !BOOT!: track 5.26 -> 23.6 mm, vias 0 -> 3
- net LED_BUILTIN: track 0.00 -> 18.1 mm, vias 0 -> 2
- net RX1: track 0.00 -> 17.8 mm, vias 0 -> 2
- net TX1: track 0.00 -> 16.8 mm, vias 0 -> 2
- net RX2: track 15.2 -> 15.9 mm
- net I2C_!INT!: track 16.9 -> 17.5 mm
- net GND: vias 0 -> 6
