File: Hardware/MicroMod_Processor_Board-nRF52840.sch (EAGLE design)
At the start: 25 parts, among them J1 MICROMOD-2222, U1 W25QXX128MBIT-6X5, U2 MDBT50Q, Y1 32.768kHz

Commit message: Schematic updated post-proto testing
Changes made: https://docs.google.com/document/d/1057ZJf50zAkChxiBm4WqtqCuvZdJMlmnGmuK_T1RHvQ/edit
Parts:
- added D2: 1A/23V/620mV, SparkFun-DiscreteSemi:DIODE-SCHOTTKY-BAT20J
Connections:
- removed net ADC_D+: J1.G10/ADC_D+/CAM_VSYNC, U2.P0.29(AIN5)
- removed net ADC_D-: J1.G9/ADC_D-/CAM_HSYNC, U2.P0.03(AIN1)
- removed net GPIO0: J1.G0/BUS0, U2.P1.15
- removed net GPIO1: J1.G1/BUS1, U2.P1.14
- removed net SPI_!CS!1: J1.SPI_!CS!1, U2.P0.20
- removed net SPI_MISO: J1.SPI_MISO/SDIO_DATA0, U1.D0/DI, U2.P0.21
- removed net SPI_MISO1: J1.SPI_MISO1, U2.P0.02(AIN0)
- removed net SPI_MOSI: J1.SPI_MOSI/SDIO_CMD, U2.P0.14
- removed net SPI_MOSI1: J1.SPI_MOSI1, U2.P0.31(AIN7)
- new net 3.3V_EN: J1.3.3V_EN, U2.P1.15
- new net GPIO0-A: J1.G0/BUS0, U2.P0.03(AIN1)
- new net GPIO1-A: J1.G1/BUS1, U2.P0.29(AIN5)
- new net GPIO8: J1.G8, U2.P1.14
- new net N$5: D2.A, J1.3.3V
- new net SPI_!CS1!: J1.SPI_!CS1!/SDIO_DATA3, U1.D3/!HOLD!, U2.P1.00(TRACEDATA0)
- new net SPI_CIPO: J1.SPI_SDI, U2.P0.02(AIN0)
- new net SPI_CIPO1: J1.SPI_SDI1/SDIO_DATA0, U1.D1/DO, U2.P0.21
- new net SPI_COPI: J1.SPI_SDO, U2.P0.31(AIN7)
- new net SPI_COPI1: J1.SPI_SDO1/SDIO_CMD, U1.D0/DI, U2.P0.14
- net !BOOT!: now also U2.P0.07(TRACECLK); no longer U2.P0.13
- net 3.3V: now also D2.C, J1.RTC_3V; no longer J1.3.3V
- net GPIO5: now also U2.P0.17; no longer U2.P1.10
- net I2C_!INT!: now also U2.P0.15; no longer U2.P1.03
- net LED_BUILTIN: now also U2.P0.13; no longer U2.P0.07(TRACECLK)
- net RX1: now also U2.P1.10; no longer U2.P0.17
- net SDIO_DATA1: no longer U1.D1/DO
- net SPI_!CS!: now also J1.SPI_!CS!, U2.P0.20; no longer J1.SPI_!CS!/SDIO_DATA3, U1.D3/!HOLD!, U2.P1.00(TRACEDATA0)
- net SPI_SCK: now also J1.SPI_SCK, U2.P0.28(AIN4); no longer J1.SPI_SCK/SDIO_CLK, U1.CLK, U2.P0.19
- net SPI_SCK1: now also J1.SPI_SCK1/SDIO_CLK, U1.CLK, U2.P0.19; no longer J1.SPI_SCK1, U2.P0.28(AIN4)
- net TX1: now also U2.P1.03; no longer U2.P0.15
Other:
- note added: "v10"
- note removed: "v01"
- moved on the sheet: R4, R5

Commit message: Routing for v10
Connections:
- net GPIO0-A: now also U2.P0.29(AIN5); no longer U2.P0.03(AIN1)
- net GPIO1-A: now also U2.P0.03(AIN1); no longer U2.P0.29(AIN5)
Changed lines of the file:
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@@
 <net name="GPIO0-A" class="0">
+<segment>
+<pinref part="J1" gate="J1" pin="G0/BUS0"/>
+<wire x1="76.2" y1="187.96" x2="78.74" y2="187.96" width="0.1524" layer="91"/>
+<label x="78.74" y="187.96" size="1.27" layer="95" xref="yes"/>
+</segment>
+<segment>
+<pinref part="U2" gate="G$1" pin="P0.29(AIN5)"/>
+<wire x1="210.82" y1="177.8" x2="213.36" y2="177.8" width="0.1524" layer="91"/>
+<label x="213.36" y="177.8" size="1.27" layer="95" xref="yes"/>
+</segment>
+</net>
+<net name="GPIO1-A" class="0">
+<segment>
+<pinref part="J1" gate="J1" pin="G1/BUS1"/>
+<wire x1="76.2" y1="185.42" x2="78.74" y2="185.42" width="0.1524" layer="91"/>
+<label x="78.74" y="185.42" size="1.27" layer="95" xref="yes"/>
+</segment>
 <segment>
 <pinref part="U2" gate="G$1" pin="P0.03(AIN1)"/>
@@
 <label x="213.36" y="243.84" size="1.27" layer="95" xref="yes"/>
 </segment>
-<segment>
-<pinref part="J1" gate="J1" pin="G0/BUS0"/>
-<wire x1="76.2" y1="187.96" x2="78.74" y2="187.96" width="0.1524" layer="91"/>
-<label x="78.74" y="187.96" size="1.27" layer="95" xref="yes"/>
-</segment>
 </net>
-<net name="GPIO1-A" class="0">
-<segment>
-<pinref part="U2" gate="G$1" pin="P0.29(AIN5)"/>
-<wire x1="210.82" y1="177.8" x2="213.36" y2="177.8" width="0.1524" layer="91"/>
-<label x="213.36" y="177.8" size="1.27" layer="95" xref="yes"/>
-</segment>
-<segment>
-<pinref part="J1" gate="J1" pin="G1/BUS1"/>
-<wire x1="76.2" y1="185.42" x2="78.74" y2="185.42" width="0.1524" layer="91"/>
-<label x="78.74" y="185.42" size="1.27" layer="95" xref="yes"/>
-</segment>
-</net>

Commit message: Design review and checklist changes
Connections:
- net GPIO0-A renamed GPIO0/ADC2
- net GPIO1-A renamed GPIO1/ADC3
- net SPI_!CS1! renamed SPI_!CS1!/SDIO_DATA3
- net SPI_CIPO1 renamed SPI_CIPO1/SDIO_DATA0
- net SPI_COPI1 renamed SPI_COPI1/SDIO_CMD
- net SPI_SCK1 renamed SPI_SCK1/SDIO_CLK
- removed net NFC1: J1.CAN-TX, U2.P0.09(NFC1)
- removed net NFC2: J1.CAN-RX, U2.P0.10(NFC2)
- new net GPIO10/NFC2: J1.G10/ADC_D+/CAM_VSYNC, U2.P0.10(NFC2)
- new net GPIO9/NFC1: J1.G9/ADC_D-/CAM_HSYNC, U2.P0.09(NFC1)
Other:
- note added: "3V logic level"
Changed lines of the file:
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@@
 <?xml version="1.0" encoding="utf-8"?>
 <!DOCTYPE eagle SYSTEM "eagle.dtd">
-<eagle version="9.4.2">
+<eagle version="9.5.2">
 <drawing>
 <settings>
-<setting alwaysvectorfont="yes"/>
+<setting alwaysvectorfont="no"/>
 <setting verticaltext="up"/>
 </settings>
@@
 <text x="190.5" y="147.828" size="2.54" layer="96" font="vector" align="center">Voltage Range: 1.7 to 5.5V</text>
 <text x="190.754" y="268.986" size="2.54" layer="94" font="vector" align="center">nRF52840</text>
+<text x="17.78" y="264.16" size="1.778" layer="97">3V logic level</text>
 </plain>
 <instances>
@@
 </segment>
 </net>
-<net name="SPI_SCK1" class="0">
+<net name="SPI_SCK1/SDIO_CLK" class="0">
 <segment>
 <wire x1="76.2" y1="254" x2="78.74" y2="254" width="0.1524" layer="91"/>
@@
 </segment>
 </net>
-<net name="SPI_CIPO1" class="0">
+<net name="SPI_CIPO1/SDIO_DATA0" class="0">
 <segment>
 <wire x1="76.2" y1="248.92" x2="78.74" y2="248.92" width="0.1524" layer="91"/>
@@
 </segment>
 </net>
-<net name="SPI_!CS1!" class="0">
+<net name="SPI_!CS1!/SDIO_DATA3" class="0">
 <segment>
 <wire x1="76.2" y1="241.3" x2="78.74" y2="241.3" width="0.1524" layer="91"/>
@@
 </segment>
 </net>
-<net name="GPIO0-A" class="0">
+<net name="GPIO0/ADC2" class="0">
 <segment>
 <pinref part="J1" gate="J1" pin="G0/BUS0"/>
@@
 </segment>
 </net>
-<net name="GPIO1-A" class="0">
+<net name="GPIO1/ADC3" class="0">
 <segment>
 <pinref part="J1" gate="J1" pin="G1/BUS1"/>
@@
 </segment>
 </net>
-<net name="NFC1" class="0">
+<net name="GPIO9/NFC1" class="0">
 <segment>
 <pinref part="U2" gate="G$1" pin="P0.09(NFC1)"/>
@@
 </segment>
 <segment>
-<wire x1="30.48" y1="218.44" x2="27.94" y2="218.44" width="0.1524" layer="91"/>
-<label x="27.94" y="218.44" size="1.27" layer="95" rot="R180" xref="yes"/>
-<pinref part="J1" gate="J1" pin="CAN-TX"/>
-</segment>
-</net>
-<net name="NFC2" class="0">
+<pinref part="J1" gate="J1" pin="G9/ADC_D-/CAM_HSYNC"/>
+<wire x1="76.2" y1="165.1" x2="78.74" y2="165.1" width="0.1524" layer="91"/>
+<label x="78.74" y="165.1" size="1.27" layer="95" xref="yes"/>
+</segment>
+</net>
+<net name="GPIO10/NFC2" class="0">
 <segment>
 <pinref part="U2" gate="G$1" pin="P0.10(NFC2)"/>
@@
 </segment>
 <segment>
-<wire x1="30.48" y1="215.9" x2="27.94" y2="215.9" width="0.1524" layer="91"/>
-<label x="27.94" y="215.9" size="1.27" layer="95" rot="R180" xref="yes"/>
-<pinref part="J1" gate="J1" pin="CAN-RX"/>
+<pinref part="J1" gate="J1" pin="G10/ADC_D+/CAM_VSYNC"/>
+<wire x1="76.2" y1="162.56" x2="78.74" y2="162.56" width="0.1524" layer="91"/>
+<label x="78.74" y="162.56" size="1.27" layer="95" xref="yes"/>
 </segment>
 </net>
@@
 </segment>
 </net>
-<net name="SPI_COPI1" class="0">
+<net name="SPI_COPI1/SDIO_CMD" class="0">
 <segment>
 <wire x1="76.2" y1="251.46" x2="78.74" y2="251.46" width="0.1524" layer="91"/>
